Commit message: working script just need to add mqtt stuff

File: ur_e_description/urdf/ur5e_robot.urdf.xacro (robot description, xacro)
@@ -28,5 +28,5 @@
     <parent link="world" />
     <child link = "base_link" />
-    <origin xyz="0.25 0.25 0.07" rpy="0.0 0.0 ${pi}" />
+    <origin xyz="0.2 0.3 0.08" rpy="0.0 0.0 ${pi}" />
   </joint>
 	<link name="vibrator">
